File: Propulsion/Cartemoteur.brd (EAGLE design)
At the start: 160 x 100 mm, 34 parts, among them IC1 STM32F042C6T6, IC2 MCP2562-E_SN, IC3 BD62321HFP-TR, IC4 BD62321HFP-TR, IC5 ZLDO1117G33TA, J1 43650-0400, J10 43650-0200, J11 43650-0200, J12 M20-8760542, J2 43650-0400, J3 43650-0400, J4 43650-0400, J5 43650-0200, J6 43650-0200, J7 43650-0200, J8 43650-0200, J9 43650-0200

Commit message: BOARD V1
Parts:
- added J13: MOTG, OUTech:43650-0200
- added J14: MOTD, OUTech:43650-0200
- added J15: 12V, OUTech:43650-0200
- J1, J2: value 43650-0400 -> CAN
- J10, J5, J6: value 43650-0200 -> 24V
- J11, J7: value 43650-0200 -> 12V
- J3: value 43650-0400 -> CODD
- J4: value 43650-0400 -> CODG
- J8, J9: value 43650-0200 -> 5V
- moved J9 117.7 mm to (54.6, 10.2)
- moved C15 115.9 mm to (50.8, 19.1), turned to 90 degrees
- moved C7 108.7 mm to (38.1, 19.1), turned to 90 degrees
- moved C6 99.4 mm to (34.3, 19.1), turned to 90 degrees
- moved IC5 98.9 mm to (45.1, 15.9), turned to 180 degrees
- moved J8 95.1 mm to (43.2, 10.2)
- moved C11 93.8 mm to (40.0, 21.6), turned to 270 degrees
- moved J5 92.7 mm to (40.6, 57.1), turned to 180 degrees
- moved J11 91.8 mm to (59.1, 45.1), turned to 90 degrees
- moved J7 91.7 mm to (59.1, 34.3), turned to 90 degrees
- moved C14 87.9 mm to (26.0, 20.3), turned to 180 degrees
- moved R1 86.8 mm to (14.0, 23.5), turned to 90 degrees
- moved J3 83.8 mm to (26.7, 6.35)
- moved C5 81.3 mm to (36.2, 19.1), turned to 90 degrees
- moved J12 80.9 mm to (43.8, 38.7), turned to 90 degrees
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Connections:
- removed net N$88: IC4.1
- net +12V: now also J15.1
- net +24V: now also IC4.1
- net CAN_H: now also J1.2, J2.2; no longer J1.3, J2.3
- net CAN_L: now also J1.3, J2.3; no longer J1.2, J2.2
- net GNDA: now also J15.2
- net OUT1_D: now also J14.2
- net OUT1_G: now also J13.2
- net OUT2_D: now also J14.1
- net OUT2_G: now also J13.1
Routing:
- net +3V3: track 0.00 -> 106.7 mm
- net +5V: track 0.00 -> 106.6 mm
- net +24V: track 0.00 -> 72.7 mm, vias 0 -> 2
- net RIN_D: track 0.00 -> 36.1 mm, vias 0 -> 2
- net FIN_D: track 0.00 -> 35.4 mm, vias 0 -> 2
- net NRST: track 0.00 -> 30.7 mm, vias 0 -> 2
- net SWDCLK: track 0.00 -> 30.3 mm, vias 0 -> 2
- net A_G: track 0.00 -> 29.5 mm, vias 0 -> 1
- net +12V: track 0.00 -> 29.4 mm
- net CAN_L: track 0.00 -> 27.5 mm, vias 0 -> 1
- net B_G: track 0.00 -> 26.6 mm, vias 0 -> 1
- net CAN_H: track 0.00 -> 26.3 mm
- net FIN_G: track 0.00 -> 26.2 mm, vias 0 -> 2
- net DBG_RX: track 0.00 -> 26.0 mm, vias 0 -> 2
- net RIN_G: track 0.00 -> 25.9 mm, vias 0 -> 2
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- added copper zone on layer 1, net GNDA
- added copper zone on layer 16, net GNDA
Other:
- board size 160 x 100 mm -> 67.9 x 66.3 mm
